File: lora-helium-moisture-sensor/lora_helium_moisture_sensor/lora_helium_moisture_sensor.kicad_sch (KiCad schematic)
At the start: 8 parts, among them J1 Screw_Terminal_01x02, J2 Conn_01x04_Male, U1 LM358

Commit message: complete prototype set
Other:
- note added: "link : https://www.alibaba.com/product-detail/Heltec-2020-SX1276-wireless-stick-lite_1600184492991.html"
Changed lines of the file:
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@@
   (no_connect (at 97.79 76.2))
   (no_connect (at 97.79 78.74))
+  (no_connect (at 97.79 101.6))
   (no_connect (at 97.79 88.9))
   (no_connect (at 97.79 91.44))
@@
   (no_connect (at 97.79 96.52))
   (no_connect (at 97.79 99.06))
-  (no_connect (at 97.79 101.6))
   (wire (pts (xy 156.21 64.77) (xy 156.21 69.85))
     (stroke (width 0) (type default) (color 0 0 0 0))
@@
     (effects (font (size 1.27 1.27)) (justify left bottom))
   )
-  (text "HELTEC WIRELESS STICK LITE" (at 88.9 31.115 0)
+  (text "HELTEC WIRELESS STICK LITE" (at 88.9 25.4 0)
     (effects (font (size 3 3)) (justify left bottom))
   )
@@
     (effects (font (size 1.27 1.27)) (justify left bottom))
   )
+  (text "link : https://www.alibaba.com/product-detail/Heltec-2020-SX1276-wireless-stick-lite_1600184492991.html"
+    (at 173.99 27.94 0)
+    (effects (font (size 1.27 1.27)) (justify right bottom))
+  )
   (label "DHT11" (at 81.28 123.19 0)

Commit message: complete project prototype
Parts:
- gave numbers to parts that had none: 1
Changed lines of the file:
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@@
   (symbol (lib_id "GCL_Modules&Devboards:HELTEC_WIRELESS_STICK_LITE") (at 119.38 49.53 0) (unit 1)
     (in_bom yes) (on_board yes)
-    (property "Reference" "U?" (id 0) (at 115.57 88.9 90)
+    (property "Reference" "U2" (id 0) (at 115.57 88.9 90)
       (effects (font (size 1.27 1.27)) (justify left))
     )
@@
     )
     (path "/405f6d9d-5db6-41d3-9959-949cc714120a"
-      (reference "U?") (unit 1) (value "HELTEC_WIRELESS_STICK_LITE") (footprint "")
-    )
-  )
+      (reference "U2") (unit 1) (value "HELTEC_WIRELESS_STICK_LITE") (footprint "")
+    )
+  )
